File: Hardware/FaultyCat.kicad_sch (KiCad schematic)
At the start: 92 parts, among them J1 Antenna, J10 TRIGGER_VREF, J2 BG306-02-A-2-0400-L-G, J3 Conn_01x10, J4 Header 2, J5 Header 4, J6 Input Power:2x AA Battery, J7 GLITCHER_EN, J8 ANALOG_PINS, J9 TRIGGER_IN, P1 USB_C_Plug_USB2.0, Q1 AO3422, Q2 AO3422, Q3 LDA111STR, Q4 RGT16BM65DTL, Q5 DMG3415U-7, Q7 IRLML2502, Q8 IRF7807PBF, SW1 TL3305AF260QG, SW2 ON, SW3 TL3305AF260QG, SW4 RESET, SW5 BOOT, SW6 TL3305AF260QG, SW7 SW_SP3T, T1 ATB322524, T2 ATB322524, U1 AP2112K-3.3, U2 W25Q16JV, U3 RP2040, U4 TXS0108EPW, U5 TLV75718PDBV, U6 SN74LVC1T45DBV, Y1 12Mhz

Commit message: fix(Hw):C23_And_C24_Added
Parts:
- added C23, C24: 10uF, Capacitor_SMD:C_0402_1005Metric, symbol Device:C_Small
Connections:
- net +1V8: now also C23.1
- net GND: now also C23.2, C24.2
- net VIN: now also C24.1

Commit message: Fixed shorting resistors for CAN & RS485
Parts:
- renumbered C22 to C10, C21 to C11, C8 to C12, C10 to C13, C9 to C14, C11 to C15, C12 to C16, C13 to C17, C14 to C18, C15 to C19, C16 to C20, C17 to C21, C18 to C22, C19 to C23, C20 to C24, C5 to C4, C4 to C5, C24 to C7, C23 to C8, C7 to C9, D6 to D4, D4 to D5, D5 to D6, J7 to J1, J6 to J10, J8 to J2, J9 to J3, J10 to J4, J1 to J5, J2 to J6, J3 to J7, J4 to J8, J5 to J9, Q5 to Q3, Q3 to Q4, Q4 to Q5, Q7 to Q6, Q8 to Q7, R8 to R10, R9 to R11, R10 to R12, R11 to R13, R23 to R14, R24 to R15, R25 to R16, R26 to R17, R15 to R18, R17 to R19, R16 to R20, R18 to R21, R13 to R22, R14 to R23, R19 to R24, R20 to R25, R12 to R8, R21 to R9, SW2 to SW1, SW1 to SW2, SW7 to SW3, SW3 to SW7, U6 to U1, U1 to U2, U5 to U3, U2 to U5, U3 to U6

Commit message: Revert "Fixed shorting resistors for CAN & RS485"
This reverts commit 6a0c7b165260f2393a2555b54d0e302f1b1791b0.
Parts:
- renumbered C13 to C10, C15 to C11, C16 to C12, C17 to C13, C18 to C14, C19 to C15, C20 to C16, C21 to C17, C22 to C18, C23 to C19, C24 to C20, C11 to C21, C10 to C22, C8 to C23, C7 to C24, C5 to C4, C4 to C5, C9 to C7, C12 to C8, C14 to C9, D5 to D4, D6 to D5, D4 to D6, J5 to J1, J4 to J10, J6 to J2, J7 to J3, J8 to J4, J9 to J5, J10 to J6, J1 to J7, J2 to J8, J3 to J9, Q4 to Q3, Q5 to Q4, Q3 to Q5, Q6 to Q7, Q7 to Q8, R12 to R10, R13 to R11, R8 to R12, R22 to R13, R23 to R14, R18 to R15, R20 to R16, R19 to R17, R21 to R18, R24 to R19, R25 to R20, R9 to R21, R14 to R23, R15 to R24, R16 to R25, R17 to R26, R10 to R8, R11 to R9, SW2 to SW1, SW1 to SW2, SW7 to SW3, SW3 to SW7, U2 to U1, U5 to U2, U6 to U3, U3 to U5, U1 to U6
